Commit message: update damping

File: models/model_chopstickbot/chopstick_bot_general.urdf (robot description, URDF)
Before this commit: robot chopstick_bot, 13 links, 12 joints
Joints:
- joint world_to_base: origin xyz=0.000000 0.000000 0.300000 rpy=0.000000 0.000000 0.000000 -> xyz=0.000000 0.000000 0.330000 rpy=0.000000 0.000000 0.000000

File: models/model_phonebot/phonebot_general.urdf (robot description, URDF)
Before this commit: robot phonebot_general_6motor, 29 links, 28 joints
Joints:
- joint world_to_base: origin xyz=0.000000 0.000000 0.300000 rpy=0.000000 0.000000 0.000000 -> xyz=0.000000 0.000000 0.330000 rpy=0.000000 0.000000 0.000000
